Commit message: added joystick control for jackal0

File: multi_jackal_description/urdf/accessories.urdf.xacro (robot description, xacro)
@@ -330,4 +330,35 @@
     </xacro:unless>
   </xacro:if>
+    <!-- Mount Enabled -->
+    <!-- <xacro:if value="${tower}">
+      <xacro:camera_mount prefix="${prefix}" tilt="${tilt}"/>
+      <joint name="${prefix}_camera_mount_joint" type="fixed">
+        <origin xyz="$(optenv JACKAL_BB2_OFFSET 0 0 0)"
+                rpy="$(optenv JACKAL_BB2_RPY 0 0 0)" />
+        <parent link="${parent}" />
+        <child link="${prefix}_camera_mount" />
+      </joint>
+      <joint name="${prefix}_camera_bracket_joint" type="fixed">
+        <origin xyz="0.007 0 0.02450" rpy="0 0 0" />
+        <parent link="${prefix}_camera_beam" />
+        <child link="${prefix}_camera" />
+      </joint>
+    </xacro:if> -->
+    <!-- Mount Disabled -->
+    <!-- <xacro:unless value="${tower}">
+      <link name="${prefix}_camera_base" type="fixed"/>
+      <joint name="${prefix}_camera_base_joint" type="fixed">
+        <origin xyz="$(optenv JACKAL_BB2_OFFSET 0 0 0)"
+                rpy="$(optenv JACKAL_BB2_RPY 0 0 0)" />
+        <parent link="${parent}" />
+        <child link="${prefix}_camera_base" />
+      </joint>
+      <joint name="${prefix}_camera_joint" type="fixed">
+        <origin xyz="0 0 0.018" rpy="0 0 0" />
+        <parent link="${prefix}_camera_base" />
+        <child link="${prefix}_camera" />
+      </joint>
+    </xacro:unless>
+  </xacro:if> -->
   <!-- Fender Accessories -->
   <xacro:if value="$(optenv JACKAL_FRONT_ACCESSORY_FENDER 0)">

Commit message: changed aruco_marker texture and added global ekf parameter to main launch file

File: multi_jackal_description/urdf/accessories.urdf.xacro (robot description, xacro)
@@ -288,4 +288,5 @@
   </xacro:if>
   <!-- If enabled, generate the bumblebee2 camera payload with a tilt of 0 degrees. -->
+  <!-- <xacro:include filename="/home/nils/jackal_ws/src/dynamic_object_jackal_slam/pointgrey_camera_driver/pointgrey_camera_description/urdf/pointgrey_bumblebee2.urdf.xacro" /> -->
   <xacro:include filename="$(find pointgrey_camera_description)/urdf/pointgrey_bumblebee2.urdf.xacro" />
   <!-- If enabled, generate the bumblebee2 camera payload with a tilt of 0 degrees. -->
@@ -332,35 +333,4 @@
     </xacro:if>
   </xacro:if>
-    <!-- Mount Enabled -->
-    <!-- <xacro:if value="${tower}">
-      <xacro:camera_mount prefix="${prefix}" tilt="${tilt}"/>
-      <joint name="${prefix}_camera_mount_joint" type="fixed">
-        <origin xyz="$(optenv JACKAL_BB2_OFFSET 0 0 0)"
-                rpy="$(optenv JACKAL_BB2_RPY 0 0 0)" />
-        <parent link="${parent}" />
-        <child link="${prefix}_camera_mount" />
-      </joint>
-      <joint name="${prefix}_camera_bracket_joint" type="fixed">
-        <origin xyz="0.007 0 0.02450" rpy="0 0 0" />
-        <parent link="${prefix}_camera_beam" />
-        <child link="${prefix}_camera" />
-      </joint>
-    </xacro:if> -->
-    <!-- Mount Disabled -->
-    <!-- <xacro:unless value="${tower}">
-      <link name="${prefix}_camera_base" type="fixed"/>
-      <joint name="${prefix}_camera_base_joint" type="fixed">
-        <origin xyz="$(optenv JACKAL_BB2_OFFSET 0 0 0)"
-                rpy="$(optenv JACKAL_BB2_RPY 0 0 0)" />
-        <parent link="${parent}" />
-        <child link="${prefix}_camera_base" />
-      </joint>
-      <joint name="${prefix}_camera_joint" type="fixed">
-        <origin xyz="0 0 0.018" rpy="0 0 0" />
-        <parent link="${prefix}_camera_base" />
-        <child link="${prefix}_camera" />
-      </joint>
-    </xacro:unless>
-  </xacro:if> -->
   <!-- Fender Accessories -->
   <xacro:if value="$(optenv JACKAL_FRONT_ACCESSORY_FENDER 0)">

File: multi_jackal_description/urdf/accessories/apriltag_box.urdf.xacro (robot description, xacro)
@@ -12,11 +12,25 @@
       <geometry>
         <mesh filename="package://multi_jackal_description/meshes/apriltags/apriltags$(arg config_id).dae" />
+      <!-- <ambient>0.1 0.1 0.1 1</ambient>
+      <diffuse>0 0 0 0</diffuse>
+      <specular>1 1 1 1</specular>
+      <emissive>0.5 0.5 0.5 1</emissive>  -->
       </geometry>
     </visual>
     <collision>
+      <!-- <ambient>0.1 0.1 0.1 1</ambient>
+      <diffuse>0 0 0 0</diffuse>
+      <specular>1 1 1 1</specular>
+      <emissive>0.5 0.5 0.5 1</emissive>  -->
       <origin xyz="0 0 0.15"/>
       <geometry>
         <box size="0.3 0.3 0.3" />
       </geometry>
+    <!-- <material>
+      <ambient>0.1 0.1 0.1 1</ambient>
+      <diffuse>0 0 0 0</diffuse>
+      <specular>1 1 1 1</specular>
+      <emissive>0.5 0.5 0.5 1</emissive>
+    </material> -->
     </collision>
   </link>
